File: germinator-pcb-board.kicad_pcb (KiCad board)
At the start: 2 copper layers, 0 parts

Commit message: Layout Step 2: Outline and Mechanical Constraints
Parts:
- added J1: Conn_01x15_Socket, Connector_PinSocket_2.54mm:PinSocket_1x15_P2.54mm_Vertical, F.Cu at (83.8, 59.7)
- added J2: Conn_01x15_Socket, Connector_PinSocket_2.54mm:PinSocket_1x15_P2.54mm_Vertical, F.Cu at (88.4, 59.7)
- added J3: Screw_Terminal_01x04, TerminalBlock:TerminalBlock_MaiXu_MX126-5.0-04P_1x04_P5.00mm, F.Cu at (67.9, 102.8)
- added J4: Screw_Terminal_01x03, TerminalBlock:TerminalBlock_MaiXu_MX126-5.0-03P_1x03_P5.00mm, F.Cu at (67.9, 62.4)
- added J5: Screw_Terminal_01x03, TerminalBlock:TerminalBlock_MaiXu_MX126-5.0-03P_1x03_P5.00mm, F.Cu at (67.9, 72.5)
- added J6: Screw_Terminal_01x03, TerminalBlock:TerminalBlock_MaiXu_MX126-5.0-03P_1x03_P5.00mm, F.Cu at (67.9, 82.6)
- added J7: Screw_Terminal_01x03, TerminalBlock:TerminalBlock_MaiXu_MX126-5.0-03P_1x03_P5.00mm, F.Cu at (67.9, 92.7)
- added R1: 4.7 K, Resistor_THT:R_Axial_DIN0207_L6.3mm_D2.5mm_P7.62mm_Horizontal, F.Cu at (65.5, 109.9)
- added R2: 10 K, Resistor_THT:R_Axial_DIN0207_L6.3mm_D2.5mm_P7.62mm_Horizontal, F.Cu at (65.5, 114.0)
- added U1: ESP32-DEVKIT-V1, germinator-pcb-board-libraries:ESP32_DEVKIT_V1, F.Cu at (139.4, 88.9)
Other:
- board outline added: 72.1 x 52.1 mm

Commit message: Layout step 3: Place Footprints
Parts:
- moved J7 100.0 mm to (166.3, 110.4), turned to 90 degrees
- moved J6 99.1 mm to (166.3, 93.9), turned to 90 degrees
- moved J5 98.5 mm to (166.3, 77.1), turned to 90 degrees
- moved J2 82.2 mm to (157.4, 104.4), turned to 180 degrees
- moved J3 56.0 mm to (112.3, 68.7), turned to -90 degrees
- moved J4 52.5 mm to (112.3, 90.4), turned to -90 degrees
- moved R1 44.6 mm to (110.0, 106.9)
- moved R2 44.6 mm to (110.0, 111.8)
- moved J1 39.2 mm to (121.9, 68.9)

Commit message: Layout step 4: Routing
Parts:
- moved R2 6.68 mm to (116.6, 110.7), turned to 180 degrees
- moved R1 6.68 mm to (116.6, 105.9), turned to 180 degrees
Routing:
- net /D15: track 0.00 -> 96.2 mm
- net /D4: track 0.00 -> 73.1 mm
- net GND: track 0.00 -> 37.9 mm, vias 0 -> 2
- net /D25: track 0.00 -> 22.4 mm
- net /D26: track 0.00 -> 19.3 mm
- net /Vcc: track 0.00 -> 5.36 mm
- net /TX2: track 0.00 -> 5.36 mm
- net /TX0: track 0.00 -> 5.36 mm
- net /RX2: track 0.00 -> 5.36 mm
- net /D5: track 0.00 -> 5.36 mm
- net /D23: track 0.00 -> 5.36 mm
- net /D22: track 0.00 -> 5.36 mm
- net /D21: track 0.00 -> 5.36 mm
- net /D2: track 0.00 -> 5.36 mm
- net /D19: track 0.00 -> 5.36 mm
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- added copper zone on B.Cu, net /Vcc
- added copper zone on F.Cu, net GND
