File: germinator-pcb-board.kicad_pcb (KiCad board)
At the start: 2 copper layers, 72.1 x 52.1 mm, 10 parts, among them J1 Conn_01x15_Socket, J2 Conn_01x15_Socket, J3 Screw_Terminal_01x04, J4 Screw_Terminal_01x03, J5 Screw_Terminal_01x03, J6 Screw_Terminal_01x03, J7 Screw_Terminal_01x03, U1 ESP32-DEVKIT-V1

Commit message: Layout step 5: Silkscreen
Parts:
- added QR*****: https://github.com/rbid/germinartor-pcb-board, germinator-pcb-board-libraries:germinartor-pcb-board-qrcode, B.Cu at (139.6, 88.1)
- added REF**: KiCad-Logo2_5mm_SilkScreen, Symbol:KiCad-Logo2_5mm_SilkScreen, B.Cu at (139.6, 102.5)
Other:
- board text added: "${ISSUE_DATE}"
- board text added: "${projectName} r ${revision}"
- board text added: "By: ${author}"
- board text added: "D12"
- board text added: "D13"
- board text added: "D14"
- board text added: "D15"
- board text added: "D18"
- board text added: "D19"
- board text added: "D2"
- board text added: "D21"
- board text added: "D22"
- board text added: "D23"
- board text added: "D25"
- board text added: "D26"
- board text added: "D27"
- board text added: "D32"
- board text added: "D33"
- board text added: "D34"
- board text added: "D35"
- board text added: "D4"
- board text added: "D5"
- board text added: "DQ"
- board text added: "Data"
- board text added: "EN"
- board text added: "GND"
- board text added: "Humidity Sensor"
- board text added: "IN1"
- board text added: "IN2"
- board text added: "RX0"
- board text added: "RX2"
- board text added: "Relays"
- board text added: "TX0"
- board text added: "TX2"
- board text added: "Temp Sensor A"
- board text added: "Temp Sensor B"
- board text added: "Temp Sensor C"
- board text added: "VIN"
- board text added: "VN"
- board text added: "VP"
- board text added: "Vcc"
