File: germinator-pcb-board.kicad_sch (KiCad schematic)
At the start: 10 parts, among them J1 Conn_01x15_Socket, J2 Conn_01x15_Socket, J3 Screw_Terminal_01x04, J4 Screw_Terminal_01x03, J5 Screw_Terminal_01x03, J6 Screw_Terminal_01x03, J7 Screw_Terminal_01x03, U1 ESP32-DEVKIT-V1

Commit message: adding terminal blocks 3d models and making traces wider
Parts:
- J4: Purpose DHT11 Humidity Sensor -> DHT11/DHT22/KY-015 Humidity Sensor
Other:
- note added: "Headers future use"
- note added: "Screw Terminal Block"
- note added: "When using a KY-015 or DHT11/DHT22 mounted on a small PCB, then the 10K pullup resistor is not needed"
- note removed: "Headers to the ESP32 for future use"
- note removed: "If using a KY-015 sensor, then there is no need to mount this pullup resistor"
Changed lines of the file:
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@@
 		(date "2025-01-23")
 		(rev "${revision}")
+		(comment 1 "Sources: ${github}")
 	)
 	(junction
@@
 		)
 	)
-	(text "Headers to the ESP32 for future use"
-		(exclude_from_sim no)
-		(at 195.58 107.95 0)
+	(text "Screw\nTerminal\nBlock"
+		(exclude_from_sim no)
+		(at 135.89 45.72 0)
+		(effects
+			(font
+				(size 1.27 1.27)
+			)
+		)
+	)
+	(text "Headers future use"
+		(exclude_from_sim no)
+		(at 186.69 107.95 0)
 		(effects
 			(font
@@
 		)
 	)
+	(text "When using a KY-015\nor DHT11/DHT22 mounted\non a small PCB, then\nthe 10K pullup resistor\nis not needed"
+		(exclude_from_sim no)
+		(at 104.14 147.32 0)
+		(effects
+			(font
+				(size 1.27 1.27)
+			)
+		)
+	)
+	(text "Screw\nTerminal\nBlock"
+		(exclude_from_sim no)
+		(at 135.89 66.04 0)
+		(effects
+			(font
+				(size 1.27 1.27)
+			)
+		)
+	)
+	(text "Screw\nTerminal\nBlock"
+		(exclude_from_sim no)
+		(at 119.38 177.8 0)
+		(effects
+			(font
+				(size 1.27 1.27)
+			)
+		)
+	)
 	(text "Relay Terminal Block"
 		(exclude_from_sim no)
@@
 		)
 	)
-	(text "If using a KY-015 sensor, then\nthere is no need to mount this\npullup resistor"
-		(exclude_from_sim no)
-		(at 102.87 147.32 0)
-		(effects
-			(font
-				(size 1.27 1.27)
-				(thickness 0.1588)
-				(italic yes)
+	(text "Screw\nTerminal\nBlock"
+		(exclude_from_sim no)
+		(at 143.51 135.89 0)
+		(effects
+			(font
+				(size 1.27 1.27)
 			)
 		)
@@
 				(thickness 0.254)
 				(bold yes)
+			)
+		)
+	)
+	(text "Screw\nTerminal\nBlock"
+		(exclude_from_sim no)
+		(at 135.89 86.36 0)
+		(effects
+			(font
+				(size 1.27 1.27)
 			)
 		)
@@
 		)
 		(property "Purpose" "DS18B20 Temp Sensor"
-			(at 129.54 60.96 0)
+			(at 129.54 59.69 0)
 			(effects
 				(font
@@
 		)
 		(property "Purpose" "DS18B20 Temp Sensor"
-			(at 129.54 81.28 0)
+			(at 129.54 80.01 0)
 			(effects
 				(font
@@
 		(dnp no)
 		(property "Reference" "J3"
-			(at 113.03 176.5299 0)
+			(at 109.22 184.15 0)
 			(effects
 				(font
@@
 				)
 				(justify left)
+				(hide yes)
 			)
 		)
@@
 		(dnp no)
 		(property "Reference" "J4"
-			(at 139.7 134.6199 0)
+			(at 135.89 140.97 0)
 			(effects
 				(font
@@
 		)
 		(property "Value" "Screw_Terminal_01x03"
-			(at 139.7 137.1599 0)
+			(at 139.7 135.89 0)
 			(effects
 				(font
@@
 				)
 				(justify left)
+				(hide yes)
 			)
 		)
@@
 			)
 		)
-		(property "Purpose" "DHT11 Humidity Sensor"
-			(at 137.16 129.54 0)
-			(effects
-				(font
+		(property "Purpose" "DHT11/DHT22/KY-015 Humidity Sensor"
+			(at 139.7 129.54 0)
+			(effects
+				(font
